File: Hardware/_Sub_HW_Mini-Scoreboard/v1_20240629/Design Folder/_HW_Mini-Scoreboard/[09] - SCATTERED LEDS.kicad_sch (KiCad schematic)
At the start: 7 parts, among them U9601 TCA9535RTWR

Commit message: Placement is done...
Parts:
- renumbered C9601 to C21401, C9602 to C21402, R9601 to R21401, R9602 to R21402, R9603 to R21403, R9604 to R21404, U9601 to U21401
Changed lines of the file:
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@@
 		(dnp no)
 		(fields_autoplaced yes)
-		(property "Reference" "#PWR09603"
+		(property "Reference" "#PWR021403"
 			(at 406.4 105.41 0)
 			(effects
@@
 		(dnp no)
 		(fields_autoplaced yes)
-		(property "Reference" "C9601"
+		(property "Reference" "C21401"
 			(at 176.53 200.6599 90)
 			(effects
@@
 		(on_board yes)
 		(dnp no)
-		(property "Reference" "R9603"
+		(property "Reference" "R21403"
 			(at 205.486 169.164 0)
 			(effects
@@
 		(dnp no)
 		(fields_autoplaced yes)
-		(property "Reference" "#PWR09601"
+		(property "Reference" "#PWR021401"
 			(at 176.53 196.85 0)
 			(effects
@@
 		(dnp no)
 		(fields_autoplaced yes)
-		(property "Reference" "C9602"
+		(property "Reference" "C21402"
 			(at 205.74 200.6599 90)
 			(effects
@@
 		(on_board yes)
 		(dnp no)
-		(property "Reference" "R9601"
+		(property "Reference" "R21401"
 			(at 205.486 145.034 0)
 			(effects
@@
 		(dnp no)
 		(fields_autoplaced yes)
-		(property "Reference" "U9601"
+		(property "Reference" "U21401"
 			(at 254 149.86 0)
 			(effects
@@
 		(on_board yes)
 		(dnp no)
-		(property "Reference" "R9604"
+		(property "Reference" "R21404"
 			(at 205.486 186.944 0)
 			(effects
@@
 		(dnp no)
 		(fields_autoplaced yes)
-		(property "Reference" "#PWR09602"
+		(property "Reference" "#PWR021402"
 			(at 229.87 223.52 0)
 			(effects
@@
 		(on_board yes)
 		(dnp no)
-		(property "Reference" "R9602"
+		(property "Reference" "R21402"
 			(at 205.486 157.734 0)
 			(effects

Commit message: Routing is going on...
Connections:
- net SINGLE LED/CATHODE renamed P1
- net SINGLE LED1/CATHODE renamed P2
- net SINGLE LED10/CATHODE renamed P11
- net SINGLE LED11/CATHODE renamed P12
- net SINGLE LED12/CATHODE renamed P13
- net SINGLE LED13/CATHODE renamed P14
- net SINGLE LED14/CATHODE renamed P15
- net SINGLE LED15/CATHODE renamed P16
- net SINGLE LED2/CATHODE renamed P3
- net SINGLE LED3/CATHODE renamed P4
- net SINGLE LED4/CATHODE renamed P5
- net SINGLE LED5/CATHODE renamed P6
- net SINGLE LED6/CATHODE renamed P7
- net SINGLE LED7/CATHODE renamed P8
- net SINGLE LED8/CATHODE renamed P9
- net SINGLE LED9/CATHODE renamed P10
