File: Hardware/_Sub_HW_Mini-Scoreboard/v1_20240629/Design Folder/_HW_Mini-Scoreboard/_HW_Mini-Scoreboard.kicad_sch (KiCad schematic)
At the start: 0 parts

Commit message: More work on the PCB....
Other:
- added sheet MECHANICAL PARTS ([12] - MECHANICAL PARTS.kicad_sch)
Changed lines of the file:
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@@
+	)
+	(sheet
+		(at 177.8 118.11)
+		(size 63.5 6.35)
+		(fields_autoplaced yes)
+		(stroke
+			(width 0.1524)
+			(type solid)
+		)
+		(fill
+			(color 0 0 0 0.0000)
+		)
+		(property "Sheetname" "MECHANICAL PARTS"
+			(at 177.8 117.3984 0)
+			(effects
+				(font
+					(size 1.27 1.27)
+				)
+				(justify left bottom)
+			)
+		)
+		(property "Sheetfile" "[12] - MECHANICAL PARTS.kicad_sch"
+			(at 177.8 125.0446 0)
+			(effects
+				(font
+					(size 1.27 1.27)
+				)
+				(justify left top)
+			)
+		)
+		(instances
+			(project "_HW_Mini-Scoreboard"
+				(path "/d8b9b213-6982-4461-908c-72226e9b7d64"
+					(page "246")
+				)
+			)
+		)
 	)
 	(sheet

Commit message: Working on bottom layer...
Other:
- removed sheet BIG 7SEGMENT
- removed sheet MEDIUM 7SEGMENT
- removed sheet SCATTERED LEDS
- removed sheet SMALL 7SEGMENT
Changed lines of the file:
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@@
-	)
-	(sheet
-		(at 63.5 194.31)
-		(size 63.5 6.35)
-		(fields_autoplaced yes)
-		(stroke
-			(width 0.1524)
-			(type solid)
-		)
-		(fill
-			(color 0 0 0 0.0000)
-		)
-		(property "Sheetname" "BIG 7SEGMENT"
-			(at 63.5 193.5984 0)
-			(effects
-				(font
-					(size 1.27 1.27)
-				)
-				(justify left bottom)
-			)
-		)
-		(property "Sheetfile" "[08] - BIG 7SEGMENT.kicad_sch"
-			(at 63.5 201.2446 0)
-			(effects
-				(font
-					(size 1.27 1.27)
-				)
-				(justify left top)
-			)
-		)
-		(instances
-			(project "_HW_Mini-Scoreboard"
-				(path "/d8b9b213-6982-4461-908c-72226e9b7d64"
-					(page "8")
-				)
-			)
-		)
-	)
-	(sheet
-		(at 63.5 168.91)
-		(size 63.5 6.35)
-		(fields_autoplaced yes)
-		(stroke
-			(width 0.1524)
-			(type solid)
-		)
-		(fill
-			(color 0 0 0 0.0000)
-		)
-		(property "Sheetname" "SMALL 7SEGMENT"
-			(at 63.5 168.1984 0)
-			(effects
-				(font
-					(size 1.27 1.27)
-				)
-				(justify left bottom)
-			)
-		)
-		(property "Sheetfile" "[06] - SMALL 7SEGMENT.kicad_sch"
-			(at 63.5 175.8446 0)
-			(effects
-				(font
-					(size 1.27 1.27)
-				)
-				(justify left top)
-			)
-		)
-		(instances
-			(project "_HW_Mini-Scoreboard"
-				(path "/d8b9b213-6982-4461-908c-72226e9b7d64"
-					(page "6")
-				)
-			)
-		)
-	)
-	(sheet
-		(at 63.5 207.01)
-		(size 63.5 6.35)
-		(fields_autoplaced yes)
-		(stroke
-			(width 0.1524)
-			(type solid)
-		)
-		(fill
-			(color 0 0 0 0.0000)
-		)
-		(property "Sheetname" "SCATTERED LEDS"
-			(at 63.5 206.2984 0)
-			(effects
-				(font
-					(size 1.27 1.27)
-				)
-				(justify left bottom)
-			)
-		)
-		(property "Sheetfile" "[09] - SCATTERED LEDS.kicad_sch"
-			(at 63.5 213.9446 0)
-			(effects
-				(font
-					(size 1.27 1.27)
-				)
-				(justify left top)
-			)
-		)
-		(instances
-			(project "_HW_Mini-Scoreboard"
-				(path "/d8b9b213-6982-4461-908c-72226e9b7d64"
-					(page "96")
-				)
-			)
-		)
-	)
-	(sheet
-		(at 63.5 181.61)
-		(size 63.5 6.35)
-		(fields_autoplaced yes)
-		(stroke
-			(width 0.1524)
-			(type solid)
-		)
-		(fill
-			(color 0 0 0 0.0000)
-		)
-		(property "Sheetname" "MEDIUM 7SEGMENT"
-			(at 63.5 180.8984 0)
-			(effects
-				(font
-					(size 1.27 1.27)
-				)
-				(justify left bottom)
-			)
-		)
-		(property "Sheetfile" "[07] - MEDIUM 7SEGMENT.kicad_sch"
-			(at 63.5 188.5446 0)
-			(effects
-				(font
-					(size 1.27 1.27)
-				)
-				(justify left top)
-			)
-		)
-		(instances
-			(project "_HW_Mini-Scoreboard"
-				(path "/d8b9b213-6982-4461-908c-72226e9b7d64"
-					(page "7")
-				)
-			)
-		)
 	)
 	(sheet

Commit message: Placement is done...
Other:
- removed sheet RS485 DRIVER
Changed lines of the file:
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@@
-	)
-	(sheet
-		(at 63.5 219.71)
-		(size 63.5 6.35)
-		(fields_autoplaced yes)
-		(stroke
-			(width 0.1524)
-			(type solid)
-		)
-		(fill
-			(color 0 0 0 0.0000)
-		)
-		(property "Sheetname" "RS485 DRIVER"
-			(at 63.5 218.9984 0)
-			(effects
-				(font
-					(size 1.27 1.27)
-				)
-				(justify left bottom)
-			)
-		)
-		(property "Sheetfile" "[10] - RS485 DRIVER.kicad_sch"
-			(at 63.5 226.6446 0)
-			(effects
-				(font
-					(size 1.27 1.27)
-				)
-				(justify left top)
-			)
-		)
-		(instances
-			(project "_HW_Mini-Scoreboard"
-				(path "/d8b9b213-6982-4461-908c-72226e9b7d64"
-					(page "130")
-				)
-			)
-		)
 	)
 	(sheet

Commit message: Update _HW_Mini-Scoreboard.kicad_sch
Other:
- note removed: "SHOULD BE ADDED AFTER RELEASE"
- company: (none) -> Mend0z0
- title: (none) -> Mini-Scoreboard
