File: Hardware/_Sub_HW_Mini-Scoreboard/v1_20240629/Design Folder/_HW_Mini-Scoreboard/[04] - TIME KEEPER.kicad_sch (KiCad schematic)
At the start: 15 parts, among them J401 HDR_5X1_VERT_2.54, U401 ATMEGA328PB-MU

Commit message: More work on the PCB....
Parts:
- renumbered C404 to C401, C405 to C402, C402 to C403, C401 to C404, C403 to C405, R407 to R402, R402 to R403, R403 to R404, R404 to R405, R405 to R406, R406 to R407

Commit message: LED placement is done...
Other:
- added sheet MEDIUM 7SEGMENT2 ([07] - MEDIUM 7SEGMENT.kicad_sch)

Commit message: Some update regarding the parts
Parts:
- removed J401: HDR_5X1_VERT_2.54, Connector_PinHeader_2.54mm:PinHeader_1x05_P2.54mm_Vertical, symbol _SCHLIB_Mini-Scoreboard:CONN_HEADER_5POS_1ROW_VERT_2.54mm
- added J401: HDR_5X1_RA_2.54, Connector_PinHeader_2.54mm:PinHeader_1x05_P2.54mm_Horizontal, symbol _SCHLIB_Mini-Scoreboard:CONN_HEADER_5POS_1ROW_RA_2.54mm
Connections:
- net ATMEGA328_MISO: now also J401.2
- net ATMEGA328_MOSI: now also J401.5
- net ATMEGA328_SCK: now also J401.3
- net ATMEGA328_~{RST}: now also J401.4
- net GND: now also J401.1
Other:
- company: (none) -> Mend0z0
- title: (none) -> Mini-Scoreboard
Changed lines of the file:
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@@
 	(generator_version "8.0")
 	(paper "C")
+	(title_block
+		(title "Mini-Scoreboard")
+		(date "2024-07-11")
+		(rev "v1.0")
+		(company "Mend0z0")
+		(comment 1 "v1.0")
+		(comment 2 "PRELIMINARY")
+		(comment 3 "Siavash Taher Parvar")
+		(comment 4 "_BOM_Mini-Scoreboard_v1.0.html")
+		(comment 5 "_PCB_Mini-Scoreboard_v1.0.kicad_pcb")
+		(comment 6 "_GBR_Mini-Scoreboard_v1.0.zip")
+		(comment 7 "_ASM_Mini-Scoreboard_v1.0.html")
+		(comment 8 "n/A")
+		(comment 9 "First Release")
+	)
 	(junction
 		(at 383.54 190.5)
@@
 	)
 	(symbol
+		(lib_id "_SCHLIB_Mini-Scoreboard:CONN_HEADER_5POS_1ROW_RA_2.54mm")
+		(at 236.22 288.29 0)
+		(unit 1)
+		(exclude_from_sim no)
+		(in_bom yes)
+		(on_board yes)
+		(dnp no)
+		(fields_autoplaced yes)
+		(property "Reference" "J401"
+			(at 242.57 290.8299 0)
+			(effects
+				(font
+					(size 1.27 1.27)
+				)
+				(justify left)
+			)
+		)
+		(property "Value" "HDR_5X1_RA_2.54"
+			(at 242.57 293.3699 0)
+			(effects
+				(font
+					(size 1.27 1.27)
+				)
+				(justify left)
+			)
+		)
+		(property "Footprint" "Connector_PinHeader_2.54mm:PinHeader_1x05_P2.54mm_Horizontal"
+			(at 238.76 271.78 0)
+			(effects
+				(font
+					(size 1.27 1.27)
+				)
+				(justify left)
+				(hide yes)
+			)
+		)
+		(property "Datasheet" "https://app.adam-tech.com/products/download/data_sheet/201281/ph1rb-xx-ua-data-sheet.pdf"
+			(at 238.76 279.4 0)
+			(effects
+				(font
+					(size 1.27 1.27)
+				)
+				(justify left)
+				(hide yes)
+			)
+		)
+		(property "Description" "Connector Header Through Hole, Right Angle 5 position 0.100\" (2.54mm)"
+			(at 238.76 274.32 0)
+			(effects
+				(font
+					(size 1.27 1.27)
+				)
+				(justify left)
+				(hide yes)
+			)
+		)
+		(property "Part Number (Manufacturer)" "PH1RB-05-UA"
+			(at 238.76 266.7 0)
+			(effects
+				(font
+					(size 1.27 1.27)
+				)
+				(justify left)
+				(hide yes)
+			)
+		)
+		(property "Manufacturer" "Adam Tech"
+			(at 238.76 264.16 0)
+			(effects
+				(font
+					(size 1.27 1.27)
+				)
+				(justify left)
+				(hide yes)
+			)
+		)
+		(property "Part Number (Vendor)" "2057-PH1RB-05-UA-ND"
+			(at 238.76 269.24 0)
+			(effects
+				(font
+					(size 1.27 1.27)
+				)
+				(justify left)
+				(hide yes)
+			)
+		)
+		(property "Vendor" "Digikey"
+			(at 238.76 261.62 0)
+			(effects
+				(font
+					(size 1.27 1.27)
+				)
+				(justify left)
+				(hide yes)
+			)
+		)
+		(property "Link" "https://www.digikey.ca/en/products/detail/adam-tech/PH1RB-05-UA/9831540"
+			(at 238.76 276.86 0)
+			(effects
+				(font
+					(size 1.27 1.27)
+				)
+				(justify left)
+				(hide yes)
+			)
+		)
+		(property "Package" "Through Hole (2.54mm)"
+			(at 242.57 295.9099 0)
+			(effects
+				(font
+					(size 1.27 1.27)
+				)
+				(justify left)
+			)
+		)
+		(property "SCH CHECK" "SCH (N/A)"
+			(at 242.57 298.4499 0)
+			(effects
+				(font
+					(size 1.27 1.27)
+				)
+				(justify left)
+			)
+		)
+		(property "PCB CHECK" "PCB (N/A)"
+			(at 242.57 300.9899 0)
+			(effects
+				(font
+					(size 1.27 1.27)
+				)
+				(justify left)
+			)
+		)
+		(pin "2"
+		)
+		(pin "1"
+		)
+		(pin "4"
+		)
+		(pin "3"
+		)
+		(pin "5"
+		)
+		(instances
+			(project ""
+				(path "/d8b9b213-6982-4461-908c-72226e9b7d64/c9b0d1bc-404d-4e82-8a2e-ab8db09511da/ab14e36f-d6f5-4615-ad8e-da8358b6603d"
+					(reference "J401")
+					(unit 1)
+				)
+			)
+		)
+	)
+	(symbol
 		(lib_id "power:GND")
 		(at 436.88 237.49 270)
@@
 					(unit 1)
 				)
-			)
-		)
-	)
-	(symbol
-		(lib_id "_SCHLIB_Mini-Scoreboard:CONN_HEADER_5POS_1ROW_VERT_2.54mm")
-		(at 236.22 288.29 0)
-		(unit 1)
-		(exclude_from_sim no)
-		(in_bom yes)
-		(on_board yes)
-		(dnp no)
-		(fields_autoplaced yes)
-		(property "Reference" "J401"
-			(at 242.57 290.8299 0)
-			(effects
-				(font
-					(size 1.27 1.27)
-				)
-				(justify left)
-			)
-		)
-		(property "Value" "HDR_5X1_VERT_2.54"
-			(at 242.57 293.3699 0)
-			(effects
-				(font
-					(size 1.27 1.27)
-				)
-				(justify left)
-			)
-		)
-		(property "Footprint" "Connector_PinHeader_2.54mm:PinHeader_1x05_P2.54mm_Vertical"
-			(at 238.76 271.78 0)
-			(effects
-				(font
-					(size 1.27 1.27)
-				)
-				(justify left)
-				(hide yes)
-			)
-		)
-		(property "Datasheet" "https://app.adam-tech.com/products/download/data_sheet/201605/ph1-xx-ua-data-sheet.pdf"
-			(at 238.76 279.4 0)
-			(effects
-				(font
-					(size 1.27 1.27)
-				)
-				(justify left)
-				(hide yes)
-			)
-		)
-		(property "Description" "Connector Header Through Hole 5 position 0.100\" (2.54mm)"
-			(at 238.76 274.32 0)
-			(effects
-				(font
-					(size 1.27 1.27)
-				)
-				(justify left)
-				(hide yes)
-			)
-		)
-		(property "Part Number (Manufacturer)" "PH1-05-UA"
-			(at 238.76 266.7 0)
-			(effects
-				(font
-					(size 1.27 1.27)
-				)
-				(justify left)
-				(hide yes)
-			)
-		)
-		(property "Manufacturer" "Adam Tech"
-			(at 238.76 264.16 0)
-			(effects
-				(font
-					(size 1.27 1.27)
-				)
-				(justify left)
-				(hide yes)
-			)
-		)
-		(property "Part Number (Vendor)" "2057-PH1-05-UA-ND"
-			(at 238.76 269.24 0)
-			(effects
-				(font
-					(size 1.27 1.27)
-				)
-				(justify left)
-				(hide yes)
-			)
-		)
-		(property "Vendor" "Digikey"
-			(at 238.76 261.62 0)
-			(effects
-				(font
-					(size 1.27 1.27)
-				)
-				(justify left)
-				(hide yes)
-			)
-		)
-		(property "Link" "https://www.digikey.ca/en/products/detail/adam-tech/PH1-05-UA/9830343?s=N4IgTCBcDaIAoAkCMBaADAVhQVQIIgF0BfIA"
-			(at 238.76 276.86 0)
-			(effects
-				(font
-					(size 1.27 1.27)
-				)
-				(justify left)
-				(hide yes)
-			)
-		)
-		(property "Package" "Through Hole (2.54mm)"
-			(at 242.57 295.9099 0)
-			(effects
-				(font
-					(size 1.27 1.27)
-				)
-				(justify left)
-			)
-		)
-		(property "SCH CHECK" "SCH (N/A)"
-			(at 242.57 298.4499 0)
-			(effects
-				(font
-					(size 1.27 1.27)
-				)
-				(justify left)
-			)
-		)
-		(property "PCB CHECK" "PCB (N/A)"
-			(at 242.57 300.9899 0)
-			(effects
-				(font
-					(size 1.27 1.27)
-				)
-				(justify left)
-			)
-		)
-		(pin "3"
-		)
-		(pin "4"
-		)
-		(pin "1"
-		)
-		(pin "2"
-		)
-		(pin "5"
-		)
-		(instances
-			(project ""
-				(path "/d8b9b213-6982-4461-908c-72226e9b7d64/c9b0d1bc-404d-4e82-8a2e-ab8db09511da/ab14e36f-d6f5-4615-ad8e-da8358b6603d"
-					(reference "J401")
-					(unit 1)
-				)
