File: Hardware/_Sub_HW_Mini-Scoreboard/v1_20240629/Design Folder/_HW_Mini-Scoreboard/[05] -  MAIN BOARD.kicad_sch (KiCad schematic)
At the start: 1 part, among them J501 FHDR_20X2_VERT_2.54

Commit message: More work on the PCB....
Connections:
- net +5V: no longer names the net of J501.2
- net +5V: no longer J501.4
- no-connect marks 27 -> 29
Changed lines of the file:
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@@
 	(generator_version "8.0")
 	(paper "C")
-	(junction
-		(at 279.4 186.69)
-		(diameter 0)
-		(color 0 0 0 0)
-	)
 	(no_connect
 		(at 248.92 224.79)
@@
 	)
 	(no_connect
+		(at 264.16 189.23)
+	)
+	(no_connect
 		(at 248.92 212.09)
 	)
@@
 	)
 	(no_connect
+		(at 264.16 186.69)
+	)
+	(no_connect
 		(at 264.16 232.41)
 	)
@@
 	(wire
 		(pts
-			(xy 279.4 186.69) (xy 280.67 186.69)
-		)
-		(stroke
-			(width 0)
-			(type default)
-		)
-	)
-	(wire
-		(pts
 			(xy 280.67 222.25) (xy 264.16 222.25)
 		)
@@
 	(wire
 		(pts
-			(xy 264.16 189.23) (xy 279.4 189.23)
-		)
-		(stroke
-			(width 0)
-			(type default)
-		)
-	)
-	(wire
-		(pts
 			(xy 242.57 196.85) (xy 248.92 196.85)
 		)
@@
 	(wire
 		(pts
-			(xy 279.4 189.23) (xy 279.4 186.69)
-		)
-		(stroke
-			(width 0)
-			(type default)
-		)
-	)
-	(wire
-		(pts
 			(xy 444.5 194.31) (xy 457.2 194.31)
 		)
@@
 		(pts
 			(xy 242.57 217.17) (xy 248.92 217.17)
-		)
-		(stroke
-			(width 0)
-			(type default)
-		)
-	)
-	(wire
-		(pts
-			(xy 264.16 186.69) (xy 279.4 186.69)
 		)
 		(stroke
@@
 			)
 			(justify left)
-		)
-	)
-	(symbol
-		(lib_id "power:+5V")
-		(at 280.67 186.69 270)
-		(unit 1)
-		(exclude_from_sim no)
-		(in_bom yes)
-		(on_board yes)
-		(dnp no)
-		(fields_autoplaced yes)
-		(property "Reference" "#PWR0501"
-			(at 276.86 186.69 0)
-			(effects
-				(font
-					(size 1.27 1.27)
-				)
-				(hide yes)
-			)
-		)
-		(property "Value" "+5V"
-			(at 284.48 186.6899 90)
-			(effects
-				(font
-					(size 1.27 1.27)
-				)
-				(justify left)
-			)
-		)
-		(property "Footprint" ""
-			(at 280.67 186.69 0)
-			(effects
-				(font
-					(size 1.27 1.27)
-				)
-				(hide yes)
-			)
-		)
-		(property "Datasheet" ""
-			(at 280.67 186.69 0)
-			(effects
-				(font
-					(size 1.27 1.27)
-				)
-				(hide yes)
-			)
-		)
-		(property "Description" "Power symbol creates a global label with name \"+5V\""
-			(at 280.67 186.69 0)
-			(effects
-				(font
-					(size 1.27 1.27)
-				)
-				(hide yes)
-			)
-		)
-		(pin "1"
-		)
-		(instances
-			(project ""
-				(path "/d8b9b213-6982-4461-908c-72226e9b7d64/c9b0d1bc-404d-4e82-8a2e-ab8db09511da/5158d457-1542-4ac0-947e-48e2eb5ee55a"
-					(reference "#PWR0501")
-					(unit 1)
-				)
-			)
 		)
 	)
@@
 		(dnp no)
 		(fields_autoplaced yes)
-		(property "Reference" "#PWR0504"
+		(property "Reference" "#PWR0506"
 			(at 287.02 209.55 0)
 			(effects
@@
 			(project "_HW_Mini-Scoreboard"
 				(path "/d8b9b213-6982-4461-908c-72226e9b7d64/c9b0d1bc-404d-4e82-8a2e-ab8db09511da/5158d457-1542-4ac0-947e-48e2eb5ee55a"
-					(reference "#PWR0504")
+					(reference "#PWR0506")
 					(unit 1)
 				)
@@
 		(dnp no)
 		(fields_autoplaced yes)
-		(property "Reference" "#PWR0507"
+		(property "Reference" "#PWR0503"
 			(at 236.22 234.95 0)
 			(effects
@@
 			(project "_HW_Mini-Scoreboard"
 				(path "/d8b9b213-6982-4461-908c-72226e9b7d64/c9b0d1bc-404d-4e82-8a2e-ab8db09511da/5158d457-1542-4ac0-947e-48e2eb5ee55a"
-					(reference "#PWR0507")
+					(reference "#PWR0503")
 					(unit 1)
 				)
@@
 		(dnp no)
 		(fields_autoplaced yes)
-		(property "Reference" "#PWR0502"
+		(property "Reference" "#PWR0504"
 			(at 287.02 191.77 0)
 			(effects
@@
 			(project ""
 				(path "/d8b9b213-6982-4461-908c-72226e9b7d64/c9b0d1bc-404d-4e82-8a2e-ab8db09511da/5158d457-1542-4ac0-947e-48e2eb5ee55a"
-					(reference "#PWR0502")
+					(reference "#PWR0504")
 					(unit 1)
 				)
@@
 		(dnp no)
 		(fields_autoplaced yes)
-		(property "Reference" "#PWR0509"
+		(property "Reference" "#PWR0501"
 			(at 236.22 196.85 0)
 			(effects
@@
 			(project "_HW_Mini-Scoreboard"
 				(path "/d8b9b213-6982-4461-908c-72226e9b7d64/c9b0d1bc-404d-4e82-8a2e-ab8db09511da/5158d457-1542-4ac0-947e-48e2eb5ee55a"
-					(reference "#PWR0509")
+					(reference "#PWR0501")
 					(unit 1)
 				)
@@
 		(dnp no)
 		(fields_autoplaced yes)
-		(property "Reference" "#PWR0503"
+		(property "Reference" "#PWR0505"
 			(at 287.02 201.93 0)
 			(effects
@@
 			(project "_HW_Mini-Scoreboard"
 				(path "/d8b9b213-6982-4461-908c-72226e9b7d64/c9b0d1bc-404d-4e82-8a2e-ab8db09511da/5158d457-1542-4ac0-947e-48e2eb5ee55a"
-					(reference "#PWR0503")
+					(reference "#PWR0505")
 					(unit 1)
 				)
@@
 		(dnp no)
 		(fields_autoplaced yes)
-		(property "Reference" "#PWR0508"
+		(property "Reference" "#PWR0502"
 			(at 236.22 217.17 0)
 			(effects
@@
 			(project "_HW_Mini-Scoreboard"
 				(path "/d8b9b213-6982-4461-908c-72226e9b7d64/c9b0d1bc-404d-4e82-8a2e-ab8db09511da/5158d457-1542-4ac0-947e-48e2eb5ee55a"
-					(reference "#PWR0508")
+					(reference "#PWR0502")
 					(unit 1)
 				)
@@
 		(dnp no)
 		(fields_autoplaced yes)
-		(property "Reference" "#PWR0505"
+		(property "Reference" "#PWR0507"
 			(at 287.02 222.25 0)
 			(effects
@@
 			(project "_HW_Mini-Scoreboard"
 				(path "/d8b9b213-6982-4461-908c-72226e9b7d64/c9b0d1bc-404d-4e82-8a2e-ab8db09511da/5158d457-1542-4ac0-947e-48e2eb5ee55a"
-					(reference "#PWR0505")
+					(reference "#PWR0507")
 					(unit 1)
 				)
@@
 		(dnp no)
 		(fields_autoplaced yes)
-		(property "Reference" "#PWR0506"
+		(property "Reference" "#PWR0508"
 			(at 287.02 227.33 0)
 			(effects
@@
 			(project "_HW_Mini-Scoreboard"
 				(path "/d8b9b213-6982-4461-908c-72226e9b7d64/c9b0d1bc-404d-4e82-8a2e-ab8db09511da/5158d457-1542-4ac0-947e-48e2eb5ee55a"
-					(reference "#PWR0506")
+					(reference "#PWR0508")
 					(unit 1)
 				)

Commit message: Some update regarding the parts
Other:
- company: (none) -> Mend0z0
- title: (none) -> Mini-Scoreboard
Changed lines of the file:
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@@
 	(generator_version "8.0")
 	(paper "C")
+	(title_block
+		(title "Mini-Scoreboard")
+		(date "2024-07-11")
+		(rev "v1.0")
+		(company "Mend0z0")
+		(comment 1 "v1.0")
+		(comment 2 "PRELIMINARY")
+		(comment 3 "Siavash Taher Parvar")
+		(comment 4 "_BOM_Mini-Scoreboard_v1.0.html")
+		(comment 5 "_PCB_Mini-Scoreboard_v1.0.kicad_pcb")
+		(comment 6 "_GBR_Mini-Scoreboard_v1.0.zip")
+		(comment 7 "_ASM_Mini-Scoreboard_v1.0.html")
+		(comment 8 "n/A")
+		(comment 9 "First Release")
+	)
 	(no_connect
 		(at 248.92 224.79)
