File: Hardware/_Sub_HW_Mini-Scoreboard/v1_20240629/Design Folder/_HW_Mini-Scoreboard/[06] - SMALL 7SEGMENT.kicad_sch (KiCad schematic)
At the start: 7 parts, among them U6601 TCA9535RTWR

Commit message: More work on the PCB....
Parts:
- renumbered C18301 to C601, C18302 to C602, R18301 to R601, U6601 to U601
Changed lines of the file:
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@@
 		(dnp no)
 		(fields_autoplaced yes)
-		(property "Reference" "U6601"
+		(property "Reference" "U601"
 			(at 254 181.61 0)
 			(effects
@@
 		)
 		(instances
-			(project "_HW_Mini-Scoreboard"
+			(project ""
+				(path "/d8b9b213-6982-4461-908c-72226e9b7d64/4c68f6d5-173d-41d7-91cf-429cbb7bab02"
+					(reference "U601")
+					(unit 1)
+				)
 				(path "/d8b9b213-6982-4461-908c-72226e9b7d64/c9b0d1bc-404d-4e82-8a2e-ab8db09511da/29df82d1-e7a0-42f2-aff8-00da25d7625e/10206822-a149-4330-8f9a-a8c360483cf0"
 					(reference "U18301")
@@
 		(dnp no)
 		(fields_autoplaced yes)
-		(property "Reference" "C18301"
+		(property "Reference" "C601"
 			(at 176.53 232.4099 90)
 			(effects
@@
 		)
 		(instances
-			(project "_HW_Mini-Scoreboard"
+			(project ""
+				(path "/d8b9b213-6982-4461-908c-72226e9b7d64/4c68f6d5-173d-41d7-91cf-429cbb7bab02"
+					(reference "C601")
+					(unit 1)
+				)
 				(path "/d8b9b213-6982-4461-908c-72226e9b7d64/c9b0d1bc-404d-4e82-8a2e-ab8db09511da/29df82d1-e7a0-42f2-aff8-00da25d7625e/10206822-a149-4330-8f9a-a8c360483cf0"
 					(reference "C18301")
@@
 				(path "/d8b9b213-6982-4461-908c-72226e9b7d64/c9b0d1bc-404d-4e82-8a2e-ab8db09511da/29df82d1-e7a0-42f2-aff8-00da25d7625e/d5c898e7-40b5-447b-96a3-625890a17a59"
 					(reference "C19801")
+					(unit 1)
+				)
+				(path "/d8b9b213-6982-4461-908c-72226e9b7d64/c9b0d1bc-404d-4e82-8a2e-ab8db09511da/30e346ea-1619-4141-b4a7-269108032fc4/10206822-a149-4330-8f9a-a8c360483cf0"
+					(reference "C6601")
+					(unit 1)
+				)
+				(path "/d8b9b213-6982-4461-908c-72226e9b7d64/c9b0d1bc-404d-4e82-8a2e-ab8db09511da/30e346ea-1619-4141-b4a7-269108032fc4/d5c898e7-40b5-447b-96a3-625890a17a59"
+					(reference "C5101")
+					(unit 1)
+				)
+				(path "/d8b9b213-6982-4461-908c-72226e9b7d64/c9b0d1bc-404d-4e82-8a2e-ab8db09511da/ab14e36f-d6f5-4615-ad8e-da8358b6603d/194c4001-596c-4389-a1ba-f1d31cb2d4b6"
+					(reference "C14701")
 					(unit 1)
 				)
@@
 		(dnp no)
 		(fields_autoplaced yes)
-		(property "Reference" "#PWR0602"
+		(property "Reference" "#PWR0601"
 			(at 176.53 228.6 0)
 			(effects
@@
 			(project "_HW_Mini-Scoreboard"
 				(path "/d8b9b213-6982-4461-908c-72226e9b7d64/4c68f6d5-173d-41d7-91cf-429cbb7bab02"
-					(reference "#PWR0602")
+					(reference "#PWR0601")
 					(unit 1)
 				)
@@
 		(dnp no)
 		(fields_autoplaced yes)
-		(property "Reference" "C18302"
+		(property "Reference" "C602"
 			(at 205.74 232.4099 90)
 			(effects
@@
 		)
 		(instances
-			(project "_HW_Mini-Scoreboard"
+			(project ""
+				(path "/d8b9b213-6982-4461-908c-72226e9b7d64/4c68f6d5-173d-41d7-91cf-429cbb7bab02"
+					(reference "C602")
+					(unit 1)
+				)
 				(path "/d8b9b213-6982-4461-908c-72226e9b7d64/c9b0d1bc-404d-4e82-8a2e-ab8db09511da/29df82d1-e7a0-42f2-aff8-00da25d7625e/10206822-a149-4330-8f9a-a8c360483cf0"
 					(reference "C18302")
@@
 				(path "/d8b9b213-6982-4461-908c-72226e9b7d64/c9b0d1bc-404d-4e82-8a2e-ab8db09511da/29df82d1-e7a0-42f2-aff8-00da25d7625e/d5c898e7-40b5-447b-96a3-625890a17a59"
 					(reference "C19802")
+					(unit 1)
+				)
+				(path "/d8b9b213-6982-4461-908c-72226e9b7d64/c9b0d1bc-404d-4e82-8a2e-ab8db09511da/30e346ea-1619-4141-b4a7-269108032fc4/10206822-a149-4330-8f9a-a8c360483cf0"
+					(reference "C6602")
+					(unit 1)
+				)
+				(path "/d8b9b213-6982-4461-908c-72226e9b7d64/c9b0d1bc-404d-4e82-8a2e-ab8db09511da/30e346ea-1619-4141-b4a7-269108032fc4/d5c898e7-40b5-447b-96a3-625890a17a59"
+					(reference "C5102")
+					(unit 1)
+				)
+				(path "/d8b9b213-6982-4461-908c-72226e9b7d64/c9b0d1bc-404d-4e82-8a2e-ab8db09511da/ab14e36f-d6f5-4615-ad8e-da8358b6603d/194c4001-596c-4389-a1ba-f1d31cb2d4b6"
+					(reference "C14702")
 					(unit 1)
 				)
@@
 		(on_board yes)
 		(dnp no)
-		(property "Reference" "R18301"
+		(property "Reference" "R601"
 			(at 205.486 176.784 0)
 			(effects
@@
 		)
 		(instances
-			(project "_HW_Mini-Scoreboard"
+			(project ""
+				(path "/d8b9b213-6982-4461-908c-72226e9b7d64/4c68f6d5-173d-41d7-91cf-429cbb7bab02"
+					(reference "R601")
+					(unit 1)
+				)
 				(path "/d8b9b213-6982-4461-908c-72226e9b7d64/c9b0d1bc-404d-4e82-8a2e-ab8db09511da/29df82d1-e7a0-42f2-aff8-00da25d7625e/10206822-a149-4330-8f9a-a8c360483cf0"
 					(reference "R18301")
@@
 				(path "/d8b9b213-6982-4461-908c-72226e9b7d64/c9b0d1bc-404d-4e82-8a2e-ab8db09511da/29df82d1-e7a0-42f2-aff8-00da25d7625e/d5c898e7-40b5-447b-96a3-625890a17a59"
 					(reference "R19801")
+					(unit 1)
+				)
+				(path "/d8b9b213-6982-4461-908c-72226e9b7d64/c9b0d1bc-404d-4e82-8a2e-ab8db09511da/30e346ea-1619-4141-b4a7-269108032fc4/10206822-a149-4330-8f9a-a8c360483cf0"
+					(reference "R6601")
+					(unit 1)
+				)
+				(path "/d8b9b213-6982-4461-908c-72226e9b7d64/c9b0d1bc-404d-4e82-8a2e-ab8db09511da/30e346ea-1619-4141-b4a7-269108032fc4/d5c898e7-40b5-447b-96a3-625890a17a59"
+					(reference "R5101")
+					(unit 1)
+				)
+				(path "/d8b9b213-6982-4461-908c-72226e9b7d64/c9b0d1bc-404d-4e82-8a2e-ab8db09511da/ab14e36f-d6f5-4615-ad8e-da8358b6603d/194c4001-596c-4389-a1ba-f1d31cb2d4b6"
+					(reference "R14701")
 					(unit 1)
 				)
@@
 		(dnp no)
 		(fields_autoplaced yes)
-		(property "Reference" "#PWR0603"
+		(property "Reference" "#PWR0602"
 			(at 229.87 255.27 0)
 			(effects
@@
 			(project "_HW_Mini-Scoreboard"
 				(path "/d8b9b213-6982-4461-908c-72226e9b7d64/4c68f6d5-173d-41d7-91cf-429cbb7bab02"
-					(reference "#PWR0603")
+					(reference "#PWR0602")
 					(unit 1)
 				)
@@
 		(dnp no)
 		(fields_autoplaced yes)
-		(property "Reference" "#PWR06603"
+		(property "Reference" "#PWR0603"
 			(at 381 125.73 0)
 			(effects
@@
 		)
 		(instances
-			(project "_HW_Mini-Scoreboard"
+			(project ""
+				(path "/d8b9b213-6982-4461-908c-72226e9b7d64/4c68f6d5-173d-41d7-91cf-429cbb7bab02"
+					(reference "#PWR0603")
+					(unit 1)
+				)
 				(path "/d8b9b213-6982-4461-908c-72226e9b7d64/c9b0d1bc-404d-4e82-8a2e-ab8db09511da/29df82d1-e7a0-42f2-aff8-00da25d7625e/10206822-a149-4330-8f9a-a8c360483cf0"
 					(reference "#PWR018303")

Commit message: Placement is done...
Parts:
- renumbered C601 to C18301, C602 to C18302, R601 to R18301, R602 to R18302, R603 to R18303, R604 to R18304, U601 to U18301
Changed lines of the file:
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@@
 		(dnp no)
 		(fields_autoplaced yes)
-		(property "Reference" "U601"
+		(property "Reference" "U18301"
 			(at 254 181.61 0)
 			(effects
@@
 		(on_board yes)
 		(dnp no)
-		(property "Reference" "R604"
+		(property "Reference" "R18304"
 			(at 205.486 218.694 0)
 			(effects
@@
 		(on_board yes)
 		(dnp no)
-		(property "Reference" "R602"
+		(property "Reference" "R18302"
 			(at 205.486 189.484 0)
 			(effects
@@
 		(on_board yes)
 		(dnp no)
-		(property "Reference" "R603"
+		(property "Reference" "R18303"
 			(at 205.486 200.914 0)
 			(effects
@@
 		(dnp no)
 		(fields_autoplaced yes)
-		(property "Reference" "C601"
+		(property "Reference" "C18301"
 			(at 176.53 232.4099 90)
 			(effects
@@
 		(dnp no)
 		(fields_autoplaced yes)
-		(property "Reference" "#PWR0601"
+		(property "Reference" "#PWR018301"
 			(at 176.53 228.6 0)
 			(effects
@@
 		(dnp no)
 		(fields_autoplaced yes)
-		(property "Reference" "C602"
+		(property "Reference" "C18302"
 			(at 205.74 232.4099 90)
 			(effects
@@
 		(on_board yes)
 		(dnp no)
-		(property "Reference" "R601"
+		(property "Reference" "R18301"
 			(at 205.486 176.784 0)
 			(effects
@@
 		(dnp no)
 		(fields_autoplaced yes)
-		(property "Reference" "#PWR0602"
+		(property "Reference" "#PWR018302"
 			(at 229.87 255.27 0)
 			(effects
@@
 		(dnp no)
 		(fields_autoplaced yes)
-		(property "Reference" "#PWR0603"
+		(property "Reference" "#PWR018303"
 			(at 381 125.73 0)
 			(effects

Commit message: Some update regarding the parts
Other:
- company: (none) -> Mend0z0
- title: (none) -> Mini-Scoreboard
Changed lines of the file:
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@@
 	(generator_version "8.0")
 	(paper "C")
+	(title_block
+		(title "Mini-Scoreboard")
+		(date "2024-07-11")
+		(rev "v1.0")
+		(company "Mend0z0")
+		(comment 1 "v1.0")
+		(comment 2 "PRELIMINARY")
+		(comment 3 "Siavash Taher Parvar")
+		(comment 4 "_BOM_Mini-Scoreboard_v1.0.html")
+		(comment 5 "_PCB_Mini-Scoreboard_v1.0.kicad_pcb")
+		(comment 6 "_GBR_Mini-Scoreboard_v1.0.zip")
+		(comment 7 "_ASM_Mini-Scoreboard_v1.0.html")
+		(comment 8 "n/A")
+		(comment 9 "First Release")
+	)
 	(junction
 		(at 203.2 228.6)
