File: Hardware/_Sub_HW_Mini-Scoreboard/v1_20240629/Design Folder/_HW_Mini-Scoreboard/[0701] - MEDIUM SEGMENT.kicad_sch (KiCad schematic)
At the start: 7 parts

Commit message: More work on the PCB....
Parts:
- removed D2902, D2903, D2905, D2906: RED_2V_20mA, LED_SMD:LED_0805_2012Metric, symbol _SCHLIB_Mini-Scoreboard:DIODE_LED_RED_2V_20mA_624nm_LED-0805
- renumbered D2904 to D2903
Connections:
- net at D2901.1, D2903.1: now also R2901.1
Other:
- moved on the sheet: R2901

Commit message: LED placement is done...
Parts:
- renumbered D2903 to D2902, R2901 to R24801

Commit message: Placement is done...
Parts:
- renumbered D2901 to D24801, D2902 to D24802
Changed lines of the file:
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@@
 		(dnp no)
 		(fields_autoplaced yes)
-		(property "Reference" "D2901"
+		(property "Reference" "D24801"
 			(at 246.38 166.9414 90)
 			(effects
@@
 		(dnp no)
 		(fields_autoplaced yes)
-		(property "Reference" "D2902"
+		(property "Reference" "D24802"
 			(at 271.78 166.9414 90)
 			(effects

Commit message: Some update regarding the parts
Other:
- company: (none) -> Mend0z0
- title: (none) -> Mini-Scoreboard
Changed lines of the file:
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@@
 	(generator_version "8.0")
 	(paper "C")
+	(title_block
+		(title "Mini-Scoreboard")
+		(date "2024-07-11")
+		(rev "v1.0")
+		(company "Mend0z0")
+		(comment 1 "v1.0")
+		(comment 2 "PRELIMINARY")
+		(comment 3 "Siavash Taher Parvar")
+		(comment 4 "_BOM_Mini-Scoreboard_v1.0.html")
+		(comment 5 "_PCB_Mini-Scoreboard_v1.0.kicad_pcb")
+		(comment 6 "_GBR_Mini-Scoreboard_v1.0.zip")
+		(comment 7 "_ASM_Mini-Scoreboard_v1.0.html")
+		(comment 8 "n/A")
+		(comment 9 "First Release")
+	)
 	(junction
 		(at 254 190.5)
