File: Hardware/_Sub_HW_Mini-Scoreboard/v1_20240629/Design Folder/_HW_Mini-Scoreboard/[07] - MEDIUM 7SEGMENT.kicad_sch (KiCad schematic)
At the start: 7 parts, among them U701 TCA9535RTWR

Commit message: Placement is done...
Parts:
- renumbered C701 to C24701, C702 to C24702, R701 to R24701, R702 to R24702, R703 to R24703, R704 to R24704, U701 to U24701
Connections:
- no-connect marks 0 -> 2
Changed lines of the file:
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@@
 		(color 0 0 0 0)
+	)
+	(no_connect
+		(at 275.59 215.9)
+	)
+	(no_connect
+		(at 275.59 238.76)
 	)
 	(polyline
@@
 		(dnp no)
 		(fields_autoplaced yes)
-		(property "Reference" "#PWR0701"
+		(property "Reference" "#PWR024701"
 			(at 180.34 229.87 0)
 			(effects
@@
 		(on_board yes)
 		(dnp no)
-		(property "Reference" "R704"
+		(property "Reference" "R24704"
 			(at 209.296 219.964 0)
 			(effects
@@
 		(dnp no)
 		(fields_autoplaced yes)
-		(property "Reference" "C701"
+		(property "Reference" "C24701"
 			(at 180.34 233.6799 90)
 			(effects
@@
 		(on_board yes)
 		(dnp no)
-		(property "Reference" "R703"
+		(property "Reference" "R24703"
 			(at 209.296 202.184 0)
 			(effects
@@
 		(on_board yes)
 		(dnp no)
-		(property "Reference" "R702"
+		(property "Reference" "R24702"
 			(at 209.296 190.754 0)
 			(effects
@@
 		(dnp no)
 		(fields_autoplaced yes)
-		(property "Reference" "#PWR0702"
+		(property "Reference" "#PWR024702"
 			(at 233.68 256.54 0)
 			(effects
@@
 		(dnp no)
 		(fields_autoplaced yes)
-		(property "Reference" "C702"
+		(property "Reference" "C24702"
 			(at 209.55 233.6799 90)
 			(effects
@@
 		(dnp no)
 		(fields_autoplaced yes)
-		(property "Reference" "U701"
+		(property "Reference" "U24701"
 			(at 257.81 182.88 0)
 			(effects
@@
 		(on_board yes)
 		(dnp no)
-		(property "Reference" "R701"
+		(property "Reference" "R24701"
 			(at 209.296 178.054 0)
 			(effects

Commit message: Some update regarding the parts
Other:
- company: (none) -> Mend0z0
- title: (none) -> Mini-Scoreboard
Changed lines of the file:
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@@
 	(generator_version "8.0")
 	(paper "C")
+	(title_block
+		(title "Mini-Scoreboard")
+		(date "2024-07-11")
+		(rev "v1.0")
+		(company "Mend0z0")
+		(comment 1 "v1.0")
+		(comment 2 "PRELIMINARY")
+		(comment 3 "Siavash Taher Parvar")
+		(comment 4 "_BOM_Mini-Scoreboard_v1.0.html")
+		(comment 5 "_PCB_Mini-Scoreboard_v1.0.kicad_pcb")
+		(comment 6 "_GBR_Mini-Scoreboard_v1.0.zip")
+		(comment 7 "_ASM_Mini-Scoreboard_v1.0.html")
+		(comment 8 "n/A")
+		(comment 9 "First Release")
+	)
 	(junction
 		(at 393.7 196.85)
