File: Hardware/_Sub_HW_Mini-Scoreboard/v1_20240629/Design Folder/_HW_Mini-Scoreboard/[0801] - BIG SEGMENT.kicad_sch (KiCad schematic)
At the start: 13 parts, among them Q23201 BC857B,215

Commit message: More work on the PCB....
Parts:
- removed D5003, D5004, D5007, D5008: RED_2V_20mA, LED_SMD:LED_0805_2012Metric, symbol _SCHLIB_Mini-Scoreboard:DIODE_LED_RED_2V_20mA_624nm_LED-0805
- removed Q23201: BC857B,215, Package_TO_SOT_SMD:SOT-23-3, symbol _SCHLIB_Mini-Scoreboard:Q_BJT_BC857B,215_PNP_45V_0.1A_0.25W_SOT-23-3
- removed R23201, R5004: 10kR_1/10W_1%, Resistor_SMD:R_0603_1608Metric, symbol _SCHLIB_Mini-Scoreboard:RES_10kR_1/10W_1%_R0603
- removed R5002: 100R_1/8W_1%, Resistor_SMD:R_0805_2012Metric, symbol _SCHLIB_Mini-Scoreboard:RES_100R_1/8W_1%_R0805
- renumbered D5005 to D5003, D5006 to D5004, R23203 to R5003
Connections:
- net CATHODE: now also R5003.2

Commit message: LED placement is done...
Parts:
- renumbered R5003 to R5001

Commit message: Placement is done...
Parts:
- renumbered D5001 to D23201, D5002 to D23202, D5003 to D23203, D5004 to D23204, R5001 to R23201
Changed lines of the file:
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@@
 		(dnp no)
 		(fields_autoplaced yes)
-		(property "Reference" "D5002"
+		(property "Reference" "D23202"
 			(at 246.38 179.6414 90)
 			(effects
@@
 		(dnp no)
 		(fields_autoplaced yes)
-		(property "Reference" "D5001"
+		(property "Reference" "D23201"
 			(at 246.38 154.2414 90)
 			(effects
@@
 		(dnp no)
 		(fields_autoplaced yes)
-		(property "Reference" "D5004"
+		(property "Reference" "D23204"
 			(at 271.78 179.6414 90)
 			(effects
@@
 		(dnp no)
 		(fields_autoplaced yes)
-		(property "Reference" "R5001"
+		(property "Reference" "R23201"
 			(at 256.54 217.1699 90)
 			(effects
@@
 		(dnp no)
 		(fields_autoplaced yes)
-		(property "Reference" "D5003"
+		(property "Reference" "D23203"
 			(at 271.78 154.2414 90)
 			(effects

Commit message: Routing is on-going...
Connections:
- net at D23201.1, D23202.2: no longer D23203.1, D23204.2
- new net: D23203.1, D23204.2
Changed lines of the file:
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@@
 	(paper "C")
-	(junction
-		(at 241.3 171.45)
-		(diameter 0)
-		(color 0 0 0 0)
-	)
 	(junction
 		(at 254 139.7)
@@
 	(junction
 		(at 254 203.2)
-		(diameter 0)
-		(color 0 0 0 0)
-	)
-	(junction
-		(at 266.7 171.45)
 		(diameter 0)
 		(color 0 0 0 0)
@@
 	(wire
 		(pts
-			(xy 241.3 165.1) (xy 241.3 171.45)
+			(xy 241.3 165.1) (xy 241.3 177.8)
 		)
 		(stroke
@@
 	(wire
 		(pts
-			(xy 266.7 165.1) (xy 266.7 171.45)
+			(xy 266.7 165.1) (xy 266.7 177.8)
 		)
 		(stroke
@@
 	(wire
 		(pts
-			(xy 241.3 171.45) (xy 266.7 171.45)
-		)
-		(stroke
-			(width 0)
-			(type default)
-		)
-	)
-	(wire
-		(pts
-			(xy 241.3 177.8) (xy 241.3 171.45)
-		)
-		(stroke
-			(width 0)
-			(type default)
-		)
-	)
-	(wire
-		(pts
 			(xy 241.3 152.4) (xy 241.3 139.7)
 		)
 		(stroke
-			(width 0)
-			(type default)
-		)
-	)
-	(wire
-		(pts
-			(xy 266.7 171.45) (xy 266.7 177.8)
-		)
-		(stroke

Commit message: Some update regarding the parts
Other:
- company: (none) -> Mend0z0
- title: (none) -> Mini-Scoreboard
Changed lines of the file:
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@@
 	(generator_version "8.0")
 	(paper "C")
+	(title_block
+		(title "Mini-Scoreboard")
+		(date "2024-07-11")
+		(rev "v1.0")
+		(company "Mend0z0")
+		(comment 1 "v1.0")
+		(comment 2 "PRELIMINARY")
+		(comment 3 "Siavash Taher Parvar")
+		(comment 4 "_BOM_Mini-Scoreboard_v1.0.html")
+		(comment 5 "_PCB_Mini-Scoreboard_v1.0.kicad_pcb")
+		(comment 6 "_GBR_Mini-Scoreboard_v1.0.zip")
+		(comment 7 "_ASM_Mini-Scoreboard_v1.0.html")
+		(comment 8 "n/A")
+		(comment 9 "First Release")
+	)
 	(junction
 		(at 254 139.7)
