File: Hardware/_Sub_HW_Mini-Scoreboard/v1_20240629/Design Folder/_HW_Mini-Scoreboard/[08] - BIG 7SEGMENT.kicad_sch (KiCad schematic)
At the start: 7 parts, among them U801 TCA9535RTWR

Commit message: Placement is done...
Parts:
- renumbered C801 to C23101, C802 to C23102, R801 to R23101, R802 to R23102, R803 to R23103, R804 to R23104, U801 to U23101
Changed lines of the file:
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@@
 		(dnp no)
 		(fields_autoplaced yes)
-		(property "Reference" "U801"
+		(property "Reference" "U23101"
 			(at 252.73 173.99 0)
 			(effects
@@
 		(dnp no)
 		(fields_autoplaced yes)
-		(property "Reference" "#PWR0802"
+		(property "Reference" "#PWR023102"
 			(at 228.6 247.65 0)
 			(effects
@@
 		(dnp no)
 		(fields_autoplaced yes)
-		(property "Reference" "C802"
+		(property "Reference" "C23102"
 			(at 204.47 224.7899 90)
 			(effects
@@
 		(dnp no)
 		(fields_autoplaced yes)
-		(property "Reference" "#PWR0803"
+		(property "Reference" "#PWR023103"
 			(at 419.1 114.3 0)
 			(effects
@@
 		(on_board yes)
 		(dnp no)
-		(property "Reference" "R802"
+		(property "Reference" "R23102"
 			(at 204.216 181.864 0)
 			(effects
@@
 		(on_board yes)
 		(dnp no)
-		(property "Reference" "R803"
+		(property "Reference" "R23103"
 			(at 204.216 193.294 0)
 			(effects
@@
 		(dnp no)
 		(fields_autoplaced yes)
-		(property "Reference" "#PWR0801"
+		(property "Reference" "#PWR023101"
 			(at 175.26 220.98 0)
 			(effects
@@
 		(dnp no)
 		(fields_autoplaced yes)
-		(property "Reference" "C801"
+		(property "Reference" "C23101"
 			(at 175.26 224.7899 90)
 			(effects
@@
 		(on_board yes)
 		(dnp no)
-		(property "Reference" "R801"
+		(property "Reference" "R23101"
 			(at 204.216 169.164 0)
 			(effects
@@
 		(on_board yes)
 		(dnp no)
-		(property "Reference" "R804"
+		(property "Reference" "R23104"
 			(at 204.216 211.074 0)
 			(effects

Commit message: Some update regarding the parts
Other:
- company: (none) -> Mend0z0
- title: (none) -> Mini-Scoreboard
Changed lines of the file:
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@@
 	(generator_version "8.0")
 	(paper "C")
+	(title_block
+		(title "Mini-Scoreboard")
+		(date "2024-07-11")
+		(rev "v1.0")
+		(company "Mend0z0")
+		(comment 1 "v1.0")
+		(comment 2 "PRELIMINARY")
+		(comment 3 "Siavash Taher Parvar")
+		(comment 4 "_BOM_Mini-Scoreboard_v1.0.html")
+		(comment 5 "_PCB_Mini-Scoreboard_v1.0.kicad_pcb")
+		(comment 6 "_GBR_Mini-Scoreboard_v1.0.zip")
+		(comment 7 "_ASM_Mini-Scoreboard_v1.0.html")
+		(comment 8 "n/A")
+		(comment 9 "First Release")
+	)
 	(junction
 		(at 419.1 138.43)
