File: Hardware/_Sub_HW_Mini-Scoreboard/v1_20240629/Design Folder/_HW_Mini-Scoreboard/[10] - RS485 DRIVER.kicad_sch (KiCad schematic)
At the start: 7 parts, among them U16201 TPT485N-SO1R

Commit message: More work on the PCB....
Parts:
- renumbered R21301 to R13001, R16201 to R13002, R16202 to R13003, R13003 to R13004, U16201 to U13001
Changed lines of the file:
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@@
 		(on_board yes)
 		(dnp no)
-		(property "Reference" "R13003"
+		(property "Reference" "R13004"
 			(at 205.486 175.006 0)
 			(effects
@@
 			(project "_HW_Mini-Scoreboard"
 				(path "/d8b9b213-6982-4461-908c-72226e9b7d64/d7949e1f-9227-4000-9c18-50817964fa3e"
-					(reference "R13003")
+					(reference "R13004")
 					(unit 1)
 				)
@@
 				)
 				(path "/d8b9b213-6982-4461-908c-72226e9b7d64/c9b0d1bc-404d-4e82-8a2e-ab8db09511da/30e346ea-1619-4141-b4a7-269108032fc4/56b5ce7b-aef9-43f8-8f48-55dfd4691f2d"
-					(reference "R13103")
+					(reference "R13104")
 					(unit 1)
 				)
 				(path "/d8b9b213-6982-4461-908c-72226e9b7d64/c9b0d1bc-404d-4e82-8a2e-ab8db09511da/5158d457-1542-4ac0-947e-48e2eb5ee55a/faef1fe1-2755-4de7-8640-8a1c71cb772e"
-					(reference "R18003")
+					(reference "R18004")
 					(unit 1)
 				)
 				(path "/d8b9b213-6982-4461-908c-72226e9b7d64/c9b0d1bc-404d-4e82-8a2e-ab8db09511da/ab14e36f-d6f5-4615-ad8e-da8358b6603d/1abca45b-3e3f-401e-a52d-c62afc62da6f"
-					(reference "R16203")
+					(reference "R16204")
 					(unit 1)
 				)
@@
 		(on_board yes)
 		(dnp no)
-		(property "Reference" "R16202"
+		(property "Reference" "R13003"
 			(at 205.74 167.64 0)
 			(effects
@@
 		)
 		(instances
-			(project "_HW_Mini-Scoreboard"
+			(project ""
+				(path "/d8b9b213-6982-4461-908c-72226e9b7d64/d7949e1f-9227-4000-9c18-50817964fa3e"
+					(reference "R13003")
+					(unit 1)
+				)
 				(path "/d8b9b213-6982-4461-908c-72226e9b7d64/c9b0d1bc-404d-4e82-8a2e-ab8db09511da/29df82d1-e7a0-42f2-aff8-00da25d7625e/56b5ce7b-aef9-43f8-8f48-55dfd4691f2d"
 					(reference "R21303")
 					(unit 1)
 				)
+				(path "/d8b9b213-6982-4461-908c-72226e9b7d64/c9b0d1bc-404d-4e82-8a2e-ab8db09511da/30e346ea-1619-4141-b4a7-269108032fc4/56b5ce7b-aef9-43f8-8f48-55dfd4691f2d"
+					(reference "R13103")
+					(unit 1)
+				)
 				(path "/d8b9b213-6982-4461-908c-72226e9b7d64/c9b0d1bc-404d-4e82-8a2e-ab8db09511da/5158d457-1542-4ac0-947e-48e2eb5ee55a/faef1fe1-2755-4de7-8640-8a1c71cb772e"
-					(reference "R18002")
+					(reference "R18003")
 					(unit 1)
 				)
 				(path "/d8b9b213-6982-4461-908c-72226e9b7d64/c9b0d1bc-404d-4e82-8a2e-ab8db09511da/ab14e36f-d6f5-4615-ad8e-da8358b6603d/1abca45b-3e3f-401e-a52d-c62afc62da6f"
-					(reference "R16202")
+					(reference "R16203")
 					(unit 1)
 				)
@@
 		(on_board yes)
 		(dnp no)
-		(property "Reference" "R21301"
+		(property "Reference" "R13001"
 			(at 155.956 181.61 0)
 			(effects
@@
 		)
 		(instances
-			(project "_HW_Mini-Scoreboard"
+			(project ""
+				(path "/d8b9b213-6982-4461-908c-72226e9b7d64/d7949e1f-9227-4000-9c18-50817964fa3e"
+					(reference "R13001")
+					(unit 1)
+				)
 				(path "/d8b9b213-6982-4461-908c-72226e9b7d64/c9b0d1bc-404d-4e82-8a2e-ab8db09511da/29df82d1-e7a0-42f2-aff8-00da25d7625e/56b5ce7b-aef9-43f8-8f48-55dfd4691f2d"
 					(reference "R21301")
+					(unit 1)
+				)
+				(path "/d8b9b213-6982-4461-908c-72226e9b7d64/c9b0d1bc-404d-4e82-8a2e-ab8db09511da/30e346ea-1619-4141-b4a7-269108032fc4/56b5ce7b-aef9-43f8-8f48-55dfd4691f2d"
+					(reference "R13101")
+					(unit 1)
+				)
+				(path "/d8b9b213-6982-4461-908c-72226e9b7d64/c9b0d1bc-404d-4e82-8a2e-ab8db09511da/5158d457-1542-4ac0-947e-48e2eb5ee55a/faef1fe1-2755-4de7-8640-8a1c71cb772e"
+					(reference "R18001")
+					(unit 1)
+				)
+				(path "/d8b9b213-6982-4461-908c-72226e9b7d64/c9b0d1bc-404d-4e82-8a2e-ab8db09511da/ab14e36f-d6f5-4615-ad8e-da8358b6603d/1abca45b-3e3f-401e-a52d-c62afc62da6f"
+					(reference "R16201")
 					(unit 1)
 				)
@@
 		(on_board yes)
 		(dnp no)
-		(property "Reference" "R16201"
+		(property "Reference" "R13002"
 			(at 205.486 158.496 0)
 			(effects
@@
 		)
 		(instances
-			(project "_HW_Mini-Scoreboard"
+			(project ""
+				(path "/d8b9b213-6982-4461-908c-72226e9b7d64/d7949e1f-9227-4000-9c18-50817964fa3e"
+					(reference "R13002")
+					(unit 1)
+				)
 				(path "/d8b9b213-6982-4461-908c-72226e9b7d64/c9b0d1bc-404d-4e82-8a2e-ab8db09511da/29df82d1-e7a0-42f2-aff8-00da25d7625e/56b5ce7b-aef9-43f8-8f48-55dfd4691f2d"
 					(reference "R21302")
 					(unit 1)
 				)
+				(path "/d8b9b213-6982-4461-908c-72226e9b7d64/c9b0d1bc-404d-4e82-8a2e-ab8db09511da/30e346ea-1619-4141-b4a7-269108032fc4/56b5ce7b-aef9-43f8-8f48-55dfd4691f2d"
+					(reference "R13102")
+					(unit 1)
+				)
 				(path "/d8b9b213-6982-4461-908c-72226e9b7d64/c9b0d1bc-404d-4e82-8a2e-ab8db09511da/5158d457-1542-4ac0-947e-48e2eb5ee55a/faef1fe1-2755-4de7-8640-8a1c71cb772e"
-					(reference "R18001")
+					(reference "R18002")
 					(unit 1)
 				)
 				(path "/d8b9b213-6982-4461-908c-72226e9b7d64/c9b0d1bc-404d-4e82-8a2e-ab8db09511da/ab14e36f-d6f5-4615-ad8e-da8358b6603d/1abca45b-3e3f-401e-a52d-c62afc62da6f"
-					(reference "R16201")
+					(reference "R16202")
 					(unit 1)
 				)
@@
 		(dnp no)
 		(fields_autoplaced yes)
-		(property "Reference" "U16201"
+		(property "Reference" "U13001"
 			(at 254 149.86 0)
 			(effects
@@
 		)
 		(instances
-			(project "_HW_Mini-Scoreboard"
+			(project ""
+				(path "/d8b9b213-6982-4461-908c-72226e9b7d64/d7949e1f-9227-4000-9c18-50817964fa3e"
+					(reference "U13001")
+					(unit 1)
+				)
 				(path "/d8b9b213-6982-4461-908c-72226e9b7d64/c9b0d1bc-404d-4e82-8a2e-ab8db09511da/29df82d1-e7a0-42f2-aff8-00da25d7625e/56b5ce7b-aef9-43f8-8f48-55dfd4691f2d"
 					(reference "U21301")
 					(unit 1)
 				)
+				(path "/d8b9b213-6982-4461-908c-72226e9b7d64/c9b0d1bc-404d-4e82-8a2e-ab8db09511da/30e346ea-1619-4141-b4a7-269108032fc4/56b5ce7b-aef9-43f8-8f48-55dfd4691f2d"
+					(reference "U13101")
+					(unit 1)
+				)

Commit message: Routing is on-going...
Parts:
- renumbered C13001 to C21301, C13002 to C21302, R13001 to R21301, R13002 to R21302, R13003 to R21303, R13004 to R21304, U13001 to U21301
Changed lines of the file:
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@@
 		(on_board yes)
 		(dnp no)
-		(property "Reference" "R13004"
+		(property "Reference" "R21304"
 			(at 205.486 175.006 0)
 			(effects
@@
 		(dnp no)
 		(fields_autoplaced yes)
-		(property "Reference" "C13002"
+		(property "Reference" "C21302"
 			(at 205.74 186.6899 90)
 			(effects
@@
 		(on_board yes)
 		(dnp no)
-		(property "Reference" "R13003"
+		(property "Reference" "R21303"
 			(at 205.74 167.64 0)
 			(effects
@@
 		(dnp no)
 		(fields_autoplaced yes)
-		(property "Reference" "#PWR013001"
+		(property "Reference" "#PWR021301"
 			(at 120.65 182.88 0)
 			(effects
@@
 		(on_board yes)
 		(dnp no)
-		(property "Reference" "R13001"
+		(property "Reference" "R21301"
 			(at 155.956 181.61 0)
 			(effects
@@
 		(dnp no)
 		(fields_autoplaced yes)
-		(property "Reference" "C13001"
+		(property "Reference" "C21301"
 			(at 176.53 186.6899 90)
 			(effects
@@
 		(on_board yes)
 		(dnp no)
-		(property "Reference" "R13002"
+		(property "Reference" "R21302"
 			(at 205.486 158.496 0)
 			(effects
@@
 		(dnp no)
 		(fields_autoplaced yes)
-		(property "Reference" "#PWR013002"
+		(property "Reference" "#PWR021302"
 			(at 173.99 209.55 0)
 			(effects
@@
 		(dnp no)
 		(fields_autoplaced yes)
-		(property "Reference" "U13001"
+		(property "Reference" "U21301"
 			(at 254 149.86 0)
 			(effects

Commit message: Some update regarding the parts
Other:
- company: (none) -> Mend0z0
- title: (none) -> Mini-Scoreboard
Changed lines of the file:
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@@
 	(generator_version "8.0")
 	(paper "C")
+	(title_block
+		(title "Mini-Scoreboard")
+		(date "2024-07-11")
+		(rev "v1.0")
+		(company "Mend0z0")
+		(comment 1 "v1.0")
+		(comment 2 "PRELIMINARY")
+		(comment 3 "Siavash Taher Parvar")
+		(comment 4 "_BOM_Mini-Scoreboard_v1.0.html")
+		(comment 5 "_PCB_Mini-Scoreboard_v1.0.kicad_pcb")
+		(comment 6 "_GBR_Mini-Scoreboard_v1.0.zip")
+		(comment 7 "_ASM_Mini-Scoreboard_v1.0.html")
+		(comment 8 "n/A")
+		(comment 9 "First Release")
+	)
 	(junction
 		(at 203.2 182.88)
