File: Hardware/_Sub_HW_Mini-Scoreboard/v1_20240629/Design Folder/_HW_Mini-Scoreboard/[11] - PWR - +5V.kicad_sch (KiCad schematic)
At the start: 4 parts, among them J18101 PWR_JACK_2X5.5MM_RA, J18102 HDR_3X1_VERT_2.54

Commit message: Some update regarding the parts
Parts:
- removed J18102: HDR_3X1_VERT_2.54, Connector_PinHeader_2.54mm:PinHeader_1x03_P2.54mm_Vertical, symbol _SCHLIB_Mini-Scoreboard:CONN_HEADER_3POS_1ROW_VERT_2.54mm
- added J11801: HDR_3X1_RA_2.54, Connector_PinHeader_2.54mm:PinHeader_1x03_P2.54mm_Horizontal, symbol _SCHLIB_Mini-Scoreboard:CONN_HEADER_3POS_1ROW_RA_2.54mm
Connections:
- net +5V: now also J11801.2
- net IN: now also J11801.1
Other:
- company: (none) -> Mend0z0
- title: (none) -> Mini-Scoreboard
Changed lines of the file:
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@@
 	(generator_version "8.0")
 	(paper "C")
+	(title_block
+		(title "Mini-Scoreboard")
+		(date "2024-07-11")
+		(rev "v1.0")
+		(company "Mend0z0")
+		(comment 1 "v1.0")
+		(comment 2 "PRELIMINARY")
+		(comment 3 "Siavash Taher Parvar")
+		(comment 4 "_BOM_Mini-Scoreboard_v1.0.html")
+		(comment 5 "_PCB_Mini-Scoreboard_v1.0.kicad_pcb")
+		(comment 6 "_GBR_Mini-Scoreboard_v1.0.zip")
+		(comment 7 "_ASM_Mini-Scoreboard_v1.0.html")
+		(comment 8 "n/A")
+		(comment 9 "First Release")
+	)
 	(junction
 		(at 243.84 182.88)
@@
 	)
 	(symbol
-		(lib_id "_SCHLIB_Mini-Scoreboard:CONN_HEADER_3POS_1ROW_VERT_2.54mm")
+		(lib_id "_SCHLIB_Mini-Scoreboard:CONN_HEADER_3POS_1ROW_RA_2.54mm")
 		(at 251.46 167.64 90)
 		(unit 1)
@@
 		(dnp no)
 		(fields_autoplaced yes)
-		(property "Reference" "J18102"
+		(property "Reference" "J11801"
 			(at 262.89 160.0199 90)
 			(effects
@@
 			)
 		)
-		(property "Value" "HDR_3X1_VERT_2.54"
+		(property "Value" "HDR_3X1_RA_2.54"
 			(at 262.89 162.5599 90)
 			(effects
@@
 			)
 		)
-		(property "Footprint" "Connector_PinHeader_2.54mm:PinHeader_1x03_P2.54mm_Vertical"
+		(property "Footprint" "Connector_PinHeader_2.54mm:PinHeader_1x03_P2.54mm_Horizontal"
 			(at 234.95 165.1 0)
 			(effects
@@
 			)
 		)
-		(property "Datasheet" "https://app.adam-tech.com/products/download/data_sheet/201605/ph1-xx-ua-data-sheet.pdf"
+		(property "Datasheet" "https://app.adam-tech.com/products/download/data_sheet/201281/ph1rb-xx-ua-data-sheet.pdf"
 			(at 242.57 165.1 0)
 			(effects
@@
 			)
 		)
-		(property "Description" "Connector Header Through Hole 3 position 0.100\" (2.54mm)"
+		(property "Description" "Connector Header Through Hole, Right Angle 3 position 0.100\" (2.54mm)"
 			(at 237.49 165.1 0)
 			(effects
@@
 			)
 		)
-		(property "Part Number (Manufacturer)" "PH1-03-UA"
+		(property "Part Number (Manufacturer)" "PH1RB-03-UA"
 			(at 229.87 165.1 0)
 			(effects
@@
 			)
 		)
-		(property "Part Number (Vendor)" "2057-PH1-03-UA-ND"
+		(property "Part Number (Vendor)" "2057-PH1RB-03-UA-ND"
 			(at 232.41 165.1 0)
 			(effects
@@
 			)
 		)
-		(property "Link" "https://www.digikey.ca/en/products/detail/adam-tech/PH1-03-UA/9830289?s=N4IgTCBcDaIAoAkCMBaADAZhQVQIIgF0BfIA"
+		(property "Link" "https://www.digikey.ca/en/products/detail/adam-tech/PH1RB-03-UA/9830403"
 			(at 240.03 165.1 0)
 			(effects
@@
 		(pin "2"
 		)
+		(pin "1"
+		)
 		(pin "3"
-		)
-		(pin "1"
 		)
 		(instances
 			(project ""
 				(path "/d8b9b213-6982-4461-908c-72226e9b7d64/e8df286b-44e1-41ee-b656-80cc2de69c59"
-					(reference "J18102")
+					(reference "J11801")
 					(unit 1)
 				)
